Commit message: adapted package names from turtlebot to turtle

File: turtle_description/urdf/sensors/asus_xtion_pro.urdf.xacro (robot description, xacro)
@@ -1,6 +1,6 @@
 <?xml version="1.0"?>
 <robot name="sensor_asus_xtion_pro" xmlns:xacro="http://ros.org/wiki/xacro">
-  <xacro:include filename="$(find turtlebot_description)/urdf/turtlebot_gazebo.urdf.xacro"/>
-  <xacro:include filename="$(find turtlebot_description)/urdf/turtlebot_properties.urdf.xacro"/>f.xacro"/>
+  <xacro:include filename="$(find turtle_description)/urdf/turtlebot_gazebo.urdf.xacro"/>
+  <xacro:include filename="$(find turtle_description)/urdf/turtlebot_properties.urdf.xacro"/>f.xacro"/>
   <!-- Xacro properties -->
   <xacro:property name="M_SCALE" value="0.001"/>
@@ -48,5 +48,5 @@
         <origin xyz="-0.01 0 0" rpy="${-M_PI/2} -${M_PI} ${-M_PI/2}"/>
         <geometry>
-          <mesh filename="package://turtlebot_description/meshes/sensors/asus_xtion_pro_live.dae" scale="${M_SCALE} ${M_SCALE} ${M_SCALE}"/>
+          <mesh filename="package://turtle_description/meshes/sensors/asus_xtion_pro_live.dae" scale="${M_SCALE} ${M_SCALE} ${M_SCALE}"/>
         </geometry>
       </visual>

File: turtle_description/urdf/stacks/hexagons.urdf.xacro (robot description, xacro)
@@ -4,5 +4,5 @@
  -->
 <robot name="stack_hexagons" xmlns:xacro="http://ros.org/wiki/xacro">
-  <xacro:include filename="$(find turtlebot_description)/urdf/common_properties.urdf.xacro"/>
+  <xacro:include filename="$(find turtle_description)/urdf/common_properties.urdf.xacro"/>
   <!-- Xacro properties -->
   <xacro:property name="M_SCALE" value="0.001"/>
@@ -19,5 +19,5 @@
         <origin xyz="0 0 0" rpy="0 0 0"/>
         <geometry>
-          <mesh filename="package://turtlebot_description/meshes/stacks/hexagons/pole_bottom.dae"/>
+          <mesh filename="package://turtle_description/meshes/stacks/hexagons/pole_bottom.dae"/>
         </geometry>
       </visual>
@@ -47,5 +47,5 @@
         <origin xyz="0 0 0" rpy="0 ${M_PI} 0"/>
         <geometry>
-          <mesh filename="package://turtlebot_description/meshes/stacks/hexagons/pole_middle.dae"/>
+          <mesh filename="package://turtle_description/meshes/stacks/hexagons/pole_middle.dae"/>
         </geometry>
       </visual>
@@ -75,5 +75,5 @@
         <origin xyz=" 0 0 0" rpy="0 0 0"/>
         <geometry>
-          <mesh filename="package://turtlebot_description/meshes/stacks/hexagons/pole_top.dae"/>
+          <mesh filename="package://turtle_description/meshes/stacks/hexagons/pole_top.dae"/>
         </geometry>
       </visual>
@@ -104,5 +104,5 @@
 <!--         <origin xyz="0 0 0" rpy="${-M_PI/2} ${M_PI} 0"/> -->
         <geometry>
-          <mesh filename="package://turtlebot_description/meshes/stacks/hexagons/pole_kinect.dae"/>
+          <mesh filename="package://turtle_description/meshes/stacks/hexagons/pole_kinect.dae"/>
         </geometry>
       </visual>
@@ -143,5 +143,5 @@
         <origin xyz="0 0 0" rpy="0 0 0"/>
         <geometry>
-          <mesh filename="package://turtlebot_description/meshes/stacks/hexagons/plate_bottom.dae"/>
+          <mesh filename="package://turtle_description/meshes/stacks/hexagons/plate_bottom.dae"/>
         </geometry>
       </visual>
@@ -173,5 +173,5 @@
         <origin xyz="0 0 0" rpy="0 0 0"/>
         <geometry>
-          <mesh filename="package://turtlebot_description/meshes/stacks/hexagons/plate_middle.dae"/>
+          <mesh filename="package://turtle_description/meshes/stacks/hexagons/plate_middle.dae"/>
         </geometry>
       </visual>
@@ -205,5 +205,5 @@
         <origin xyz="0 0 0" rpy="0 0 0"/>
         <geometry>
-          <mesh filename="package://turtlebot_description/meshes/stacks/hexagons/plate_top.dae"/>
+          <mesh filename="package://turtle_description/meshes/stacks/hexagons/plate_top.dae"/>
         </geometry>
       </visual>
