Commit message: modified robot model for simulator (kinect not right yet)

File: turtlebot_description/urdf/sensors/hokuyo_laser.urdf.xacro (robot description, xacro)
@@ -5,5 +5,5 @@
   <xacro:macro name="sensor_hokuyo" params="parent">
   <joint name="laser" type="fixed">
-    <origin xyz="-0.1285 0.00 0.348" rpy="0 0 0" />
+    <origin xyz="0.055 0.00 0.2254" rpy="0 0 0" />
     <parent link="${parent}" />
     <child link="base_laser_link" />

File: turtlebot_description/urdf/turtlebot_gazebo.urdf.xacro (robot description, xacro)
@@ -52,6 +52,6 @@
               <samples>720</samples>
               <resolution>1</resolution>
-              <min_angle>-1.570796</min_angle>
-              <max_angle>1.570796</max_angle>
+              <min_angle>-2.2689</min_angle>
+              <max_angle>2.2689</max_angle>
             </horizontal>
           </scan>
@@ -68,5 +68,5 @@
         </ray>
         <plugin name="hokuyo_node" filename="libgazebo_ros_laser.so">
-          <topicName>/scan</topicName>
+          <topicName>/scan_hokuyo</topicName>
           <frameName>base_laser_link</frameName>
         </plugin>

File: turtlebot_description/urdf/turtlebot_library.urdf.xacro (robot description, xacro)
@@ -7,4 +7,5 @@
   <xacro:include filename="$(find turtlebot_description)/urdf/common_properties.urdf.xacro"/>
   <xacro:include filename="$(find turtlebot_description)/urdf/turtlebot_properties.urdf.xacro"/>
+  <xacro:include filename="$(find turtlebot_description)/urdf/ninjabot_properties.urdf.xacro"/>
   <!-- Bases -->
   <xacro:include filename="$(find create_description)/urdf/create.urdf.xacro"/>
@@ -13,5 +14,7 @@
   <xacro:include filename="$(find turtlebot_description)/urdf/stacks/circles.urdf.xacro"/>
   <xacro:include filename="$(find turtlebot_description)/urdf/stacks/hexagons.urdf.xacro"/>
+  <xacro:include filename="$(find turtlebot_description)/urdf/stacks/ninja-hexagons.urdf.xacro"/>
   <!-- 3D Sensors -->
+  <xacro:include filename="$(find turtlebot_description)/urdf/sensors/ninjakinect.urdf.xacro"/>
   <xacro:include filename="$(find turtlebot_description)/urdf/sensors/kinect.urdf.xacro"/>
   <xacro:include filename="$(find turtlebot_description)/urdf/sensors/asus_xtion_pro.urdf.xacro"/>
