Commit message: fixed kinect data

File: turtlebot_description/urdf/ninjabot_properties.urdf.xacro (robot description, xacro)
@@ -20,9 +20,9 @@
      (currently in development and awaiting feedback)
    -->
-	<property name="cam_px" value="0.15" />
+	<property name="cam_px" value="0.08" />
 <!--	<property name="cam_py" value="-0.0125" /> Y varies for different configurations. get sets in sensors_urdf -->
-	<property name="cam_pz" value="0.09" />
-	<property name="cam_or" value="${-M_PI/6}" />
-	<property name="cam_op" value="${M_PI}" />
-	<property name="cam_oy" value="${M_PI/2}" />
+	<property name="cam_pz" value="0.35" />
+	<property name="cam_or" value="${M_PI}" />
+	<property name="cam_op" value="${M_PI/8}" />
+	<property name="cam_oy" value="0" />
 </robot>

File: turtlebot_description/urdf/sensors/hokuyo_laser.urdf.xacro (robot description, xacro)
@@ -2,5 +2,5 @@
 <robot name="sensor_hokuyo" xmlns:xacro="http://ros.org/wiki/xacro">
 <xacro:include filename="$(find turtlebot_description)/urdf/turtlebot_gazebo.urdf.xacro"/>
-<xacro:include filename="$(find turtlebot_description)/urdf/turtlebot_properties.urdf.xacro"/>
+<!--<xacro:include filename="$(find turtlebot_description)/urdf/turtlebot_properties.urdf.xacro"/>-->
   <xacro:macro name="sensor_hokuyo" params="parent">
   <joint name="laser" type="fixed">

File: turtlebot_description/urdf/sensors/ninjakinect.urdf.xacro (robot description, xacro)
@@ -13,5 +13,5 @@
     <link name="camera_rgb_frame"/>
     <joint name="camera_rgb_optical_joint" type="fixed">
-      <origin xyz="0 0 0" rpy="${-M_PI/2} 0 ${-M_PI/2}" />
+       <origin xyz="0 0 0" rpy="${-M_PI/2} 0 ${-M_PI/2}" /> <!--(default) -->
       <parent link="camera_rgb_frame" />
       <child link="camera_rgb_optical_frame" />
@@ -19,6 +19,5 @@
     <link name="camera_rgb_optical_frame"/>
     <joint name="camera_joint" type="fixed">
-      <!--  <origin xyz="-0.031 ${-kinect_cam_py} -0.016" rpy="0 0 0"/> -->
-     <origin xyz="0.15 0.0 0.09" rpy="${-M_PI/6} ${M_PI} ${M_PI/2}"/>
+      <origin xyz="-0.031 ${kinect_cam_py} -0.016" rpy="0 0 0"/> <!--(default) -->
       <parent link="camera_rgb_frame"/>
       <child link="camera_link"/>
@@ -26,7 +25,5 @@
       <link name="camera_link">
       <visual>
-<!--	<origin xyz="0.20 0.0 0.1" rpy="${-M_PI/6} ${M_PI} ${M_PI/2}"/> -->
-      <!-- <origin xyz="0 0 0" rpy="0 0 ${M_PI/2}"/> -->
-	<origin xyz="0 0 0" rpy="0 0 0"/>
+       <origin xyz="0 0 0" rpy="0 0 ${M_PI/2}"/>
         <geometry>
          <mesh filename="package://turtlebot_description/meshes/sensors/kinect.dae"/>
@@ -58,4 +55,5 @@
 	<joint name="camera_depth_optical_joint" type="fixed">
 	  <origin xyz="0 0 0" rpy="${-M_PI/2} 0 ${-M_PI/2}" />
+<!-- <origin xyz="0 0 0" rpy="${-M_PI/2} 0 ${-M_PI/2}" /> -->
 	  <parent link="camera_depth_frame" />
 	  <child link="camera_depth_optical_frame" />

File: turtlebot_description/urdf/turtlebot_library.urdf.xacro (robot description, xacro)
@@ -6,5 +6,5 @@
   <!-- General -->
   <xacro:include filename="$(find turtlebot_description)/urdf/common_properties.urdf.xacro"/>
-  <xacro:include filename="$(find turtlebot_description)/urdf/turtlebot_properties.urdf.xacro"/>
+<!--  <xacro:include filename="$(find turtlebot_description)/urdf/turtlebot_properties.urdf.xacro"/>-->
   <xacro:include filename="$(find turtlebot_description)/urdf/ninjabot_properties.urdf.xacro"/>
   <!-- Bases -->
@@ -17,7 +17,7 @@
   <!-- 3D Sensors -->
   <xacro:include filename="$(find turtlebot_description)/urdf/sensors/ninjakinect.urdf.xacro"/>
-  <xacro:include filename="$(find turtlebot_description)/urdf/sensors/kinect.urdf.xacro"/>
-  <xacro:include filename="$(find turtlebot_description)/urdf/sensors/asus_xtion_pro.urdf.xacro"/>
-  <xacro:include filename="$(find turtlebot_description)/urdf/sensors/asus_xtion_pro_offset.urdf.xacro"/>
+  <!--<xacro:include filename="$(find turtlebot_description)/urdf/sensors/kinect.urdf.xacro"/>-->
+<!--   <xacro:include filename="$(find turtlebot_description)/urdf/sensors/asus_xtion_pro.urdf.xacro"/>-->
+ <!--  <xacro:include filename="$(find turtlebot_description)/urdf/sensors/asus_xtion_pro_offset.urdf.xacro"/>-->
   <!-- Laser Scanner -->
   <xacro:include filename="$(find turtlebot_description)/urdf/sensors/hokuyo_laser.urdf.xacro" />
